Commit message: xacro

File: assets/player_macro.xacro (robot description, xacro)
@@ -18,6 +18,36 @@
       </inertial>
     </link>
+    <link name="${name}_x"/>
+    <link name="${name}_y"/>
     <xacro:player_foot name="${name}_right_foot"/>
     <xacro:player_foot name="${name}_left_foot"/>
+    <joint name="${name}_x_joint" type="prismatic">
+      <axis xyz="1 0 0"/>
+      <parent link="field"/>
+      <child link="${name}_x"/>
+    </joint>
+    <joint name="${name}_y_joint" type="prismatic">
+      <axis xyz="0 1 0"/>
+      <parent link="${name}_x"/>
+      <child link="${name}_y"/>
+    </joint>
+    <joint name="${name}_joint" type="continuous">
+      <axis xyz="0 0 1"/>
+      <parent link="${name}_y"/>
+      <child link="${name}"/>
+      <origin xyz="0.03 0 0.3"/>
+    </joint>
+    <joint name="${name}_right_foot_joint" type="revolute">
+      <axis xyz="0 -1 0"/>
+      <parent link="${name}"/>
+      <child link="${name}_right_foot"/>
+      <origin xyz="0.10 -0.06 0"/>
+    </joint>
+    <joint name="${name}_left_foot_joint" type="revolute">
+      <axis xyz="0 -1 0"/>
+      <parent link="${name}"/>
+      <child link="${name}_left_foot"/>
+      <origin xyz="0.10 0.06 0"/>
+    </joint>
   </xacro:macro>
   <xacro:macro name="player_foot" params="name">

Commit message: refine model

File: assets/player_macro.xacro (robot description, xacro)
@@ -3,15 +3,18 @@
     <link name="${name}">
       <visual>
+        <origin xyz="-0.015 0.000 0.300"/>
         <geometry>
-          <box size="0.14 0.2 0.6"/>
+          <box size="0.130 0.200 0.600"/>
         </geometry>
         <material name="${color}"/>
       </visual>
       <collision>
+        <origin xyz="-0.015 0.000 0.300"/>
         <geometry>
-          <box size="0.14 0.2 0.6"/>
+          <box size="0.130 0.200 0.600"/>
         </geometry>
       </collision>
       <inertial>
+        <origin xyz="-0.015 0.000 0.300"/>
         <mass value="4"/>
         <inertia ixx="0.05" ixy="0" ixz="0" iyy="0.05" iyz="0" izz="0.08"/>
@@ -36,5 +39,4 @@
       <parent link="${name}_y"/>
       <child link="${name}"/>
-      <origin xyz="0.03 0 0.3"/>
     </joint>
     <joint name="${name}_right_foot_joint" type="revolute">
@@ -42,5 +44,5 @@
       <parent link="${name}"/>
       <child link="${name}_right_foot"/>
-      <origin xyz="0.10 -0.06 0"/>
+      <origin xyz="0.070 -0.055 0.250"/>
     </joint>
     <joint name="${name}_left_foot_joint" type="revolute">
@@ -48,5 +50,5 @@
       <parent link="${name}"/>
       <child link="${name}_left_foot"/>
-      <origin xyz="0.10 0.06 0"/>
+      <origin xyz="0.070 0.055 0.250"/>
     </joint>
   </xacro:macro>
@@ -54,14 +56,14 @@
     <link name="${name}">
       <visual>
-        <origin xyz="0 0 -0.18"/>
+        <origin xyz="0.000 0.000 -0.120"/>
         <geometry>
-          <box size="0.05 0.1 0.2"/>
+          <box size="0.020 0.090 0.240"/>
         </geometry>
         <material name="yellow"/>
       </visual>
       <collision>
-        <origin xyz="0 0 -0.18"/>
+        <origin xyz="0.000 0.000 -0.120"/>
         <geometry>
-          <box size="0.05 0.1 0.2"/>
+          <box size="0.020 0.100 0.240"/>
         </geometry>
       </collision>

Commit message: fix foot size

File: assets/player_macro.xacro (robot description, xacro)
@@ -65,5 +65,5 @@
         <origin xyz="0.000 0.000 -0.120"/>
         <geometry>
-          <box size="0.020 0.100 0.240"/>
+          <box size="0.020 0.090 0.240"/>
         </geometry>
       </collision>
