Commit message: move x_y_the

File: assets/soccer.urdf (robot description, URDF)
Before this commit: robot soccer, 3 links, 2 joints
Links:
- removed link field_link
- removed link player1_link
- removed link player2_link
- added link field; visual box size=6.5 8 0.001
- added link player1, mass 5; collision box size=0.2 0.2 0.6; visual box size=0.2 0.2 0.6
- added link player1_x
- added link player1_y
Joints:
- removed joint player2_joint
- added joint player1_x_joint: type prismatic, parent field, child player1_x, axis 1 0 0
- added joint player1_y_joint: type prismatic, parent player1_x, child player1_y, axis 0 1 0
- joint player1_joint: child player1_link -> player1; parent field_link -> player1_y

Commit message: two robots

File: assets/soccer.urdf (robot description, URDF)
Before this commit: robot soccer, 4 links, 3 joints
Links:
- added link player2, mass 5; collision box size=0.2 0.2 0.6; visual box size=0.2 0.2 0.6
- added link player2_x
- added link player2_y
Joints:
- added joint player2_joint: type continuous, parent player2_y, child player2, origin xyz=0 0 0.3, axis 0 0 1
- added joint player2_x_joint: type prismatic, parent field, child player2_x, axis 1 0 0
- added joint player2_y_joint: type prismatic, parent player2_x, child player2_y, axis 0 1 0

Commit message: add red team

File: assets/soccer.urdf (robot description, URDF)
Before this commit: robot soccer, 7 links, 6 joints
Links:
- added link left_goal_post1_link; visual box size=0.10 0.10 1.2
- added link left_goal_post2_link; visual box size=0.10 0.10 1.2
- added link line1_link; visual box size=0.05 6 0.002
- added link line2_link; visual box size=9 0.05 0.002
- added link line3_link; visual box size=9 0.05 0.002
- added link line4_link; visual box size=0.05 6 0.002
- added link line5_link; visual box size=0.05 6 0.002
- added link player3, mass 5; collision box size=0.2 0.2 0.6; visual box size=0.2 0.2 0.6
- added link player3_x
- added link player3_y
- added link player4, mass 5; collision box size=0.2 0.2 0.6; visual box size=0.2 0.2 0.6
- added link player4_x
- added link player4_y
- added link right_goal_post1_link; visual box size=0.10 0.10 1.2
- added link right_goal_post2_link; visual box size=0.10 0.10 1.2
- added link top_goal_post1_link; visual box size=0.10 2.7 0.10
- added link top_goal_post2_link; visual box size=0.10 2.7 0.10
- link field: geometry visual box size=11 8 0.001
Joints:
- added joint left_goal_post1_joint: type fixed, parent field, child left_goal_post1_link, origin xyz=4.5 1.3 0.6
- added joint left_goal_post2_joint: type fixed, parent field, child left_goal_post2_link, origin xyz=-4.5 1.3 0.6
- added joint line1_joint: type fixed, parent field, child line1_link, origin xyz=4.5 0 0
- added joint line2_joint: type fixed, parent field, child line2_link, origin xyz=0 3 0
- added joint line3_joint: type fixed, parent field, child line3_link, origin xyz=0 -3 0
- added joint line4_joint: type fixed, parent field, child line4_link
- added joint line5_joint: type fixed, parent field, child line5_link, origin xyz=-4.5 0 0
- added joint player3_joint: type continuous, parent player3_y, child player3, origin xyz=0 0 0.3, axis 0 0 1
- added joint player3_x_joint: type prismatic, parent field, child player3_x, axis 1 0 0
- added joint player3_y_joint: type prismatic, parent player3_x, child player3_y, axis 0 1 0
- added joint player4_joint: type continuous, parent player4_y, child player4, origin xyz=0 0 0.3, axis 0 0 1
- added joint player4_x_joint: type prismatic, parent field, child player4_x, axis 1 0 0
- added joint player4_y_joint: type prismatic, parent player4_x, child player4_y, axis 0 1 0
- added joint right_goal_post1_joint: type fixed, parent field, child right_goal_post1_link, origin xyz=4.5 -1.3 0.6
- added joint right_goal_post2_joint: type fixed, parent field, child right_goal_post2_link, origin xyz=-4.5 -1.3 0.6
- added joint top_goal_post1_joint: type fixed, parent field, child top_goal_post1_link, origin xyz=4.5 0 1.2
- added joint top_goal_post2_joint: type fixed, parent field, child top_goal_post2_link, origin xyz=-4.5 0 1.2

Commit message: descrete

File: assets/soccer.urdf (robot description, URDF)
Before this commit: robot soccer, 24 links, 23 joints
Links:
- added link player1_left_foot, mass 0.5; collision box size=0.05 0.1 0.2; visual box size=0.05 0.1 0.2
- added link player1_right_foot, mass 0.5; collision box size=0.05 0.1 0.2; visual box size=0.05 0.1 0.2
- added link player2_left_foot, mass 0.5; collision box size=0.05 0.1 0.2; visual box size=0.05 0.1 0.2
- added link player2_right_foot, mass 0.5; collision box size=0.05 0.1 0.2; visual box size=0.05 0.1 0.2
- added link player3_left_foot, mass 0.5; collision box size=0.05 0.1 0.2; visual box size=0.05 0.1 0.2
- added link player3_right_foot, mass 0.5; collision box size=0.05 0.1 0.2; visual box size=0.05 0.1 0.2
- added link player4_left_foot, mass 0.5; collision box size=0.05 0.1 0.2; visual box size=0.05 0.1 0.2
- added link player4_right_foot, mass 0.5; collision box size=0.05 0.1 0.2; visual box size=0.05 0.1 0.2
- link player1: mass 5 -> 4; geometry collision box size=0.14 0.2 0.6; visual box size=0.14 0.2 0.6
- link player2: mass 5 -> 4; geometry collision box size=0.14 0.2 0.6; visual box size=0.14 0.2 0.6
- link player3: mass 5 -> 4; geometry collision box size=0.14 0.2 0.6; visual box size=0.14 0.2 0.6
- link player4: mass 5 -> 4; geometry collision box size=0.14 0.2 0.6; visual box size=0.14 0.2 0.6
Joints:
- added joint player1_left_foot_joint: type revolute, parent player1, child player1_left_foot, origin xyz=0.10 0.06 0, axis 0 -1 0
- added joint player1_right_foot_joint: type revolute, parent player1, child player1_right_foot, origin xyz=0.10 -0.06 0, axis 0 -1 0
- added joint player2_left_foot_joint: type revolute, parent player2, child player2_left_foot, origin xyz=0.10 0.06 0, axis 0 -1 0
- added joint player2_right_foot_joint: type revolute, parent player2, child player2_right_foot, origin xyz=0.10 -0.06 0, axis 0 -1 0
- added joint player3_left_foot_joint: type revolute, parent player3, child player3_left_foot, origin xyz=0.10 0.06 0, axis 0 -1 0
- added joint player3_right_foot_joint: type revolute, parent player3, child player3_right_foot, origin xyz=0.10 -0.06 0, axis 0 -1 0
- added joint player4_left_foot_joint: type revolute, parent player4, child player4_left_foot, origin xyz=0.10 0.06 0, axis 0 -1 0
- added joint player4_right_foot_joint: type revolute, parent player4, child player4_right_foot, origin xyz=0.10 -0.06 0, axis 0 -1 0
- joint player1_joint: origin xyz=0 0 0.3 -> xyz=0.03 0 0.3
- joint player2_joint: origin xyz=0 0 0.3 -> xyz=0.03 0 0.3
- joint player3_joint: origin xyz=0 0 0.3 -> xyz=0.03 0 0.3
- joint player4_joint: origin xyz=0 0 0.3 -> xyz=0.03 0 0.3

Commit message: variable agents

File: assets/soccer.urdf (robot description, URDF)
Before this commit: robot soccer, 32 links, 31 joints
Links:
- added link player5, mass 4; collision box size=0.14 0.2 0.6; visual box size=0.14 0.2 0.6
- added link player5_left_foot, mass 0.5; collision box size=0.05 0.1 0.2; visual box size=0.05 0.1 0.2
- added link player5_right_foot, mass 0.5; collision box size=0.05 0.1 0.2; visual box size=0.05 0.1 0.2
- added link player5_x
- added link player5_y
- added link player6, mass 4; collision box size=0.14 0.2 0.6; visual box size=0.14 0.2 0.6
- added link player6_left_foot, mass 0.5; collision box size=0.05 0.1 0.2; visual box size=0.05 0.1 0.2
- added link player6_right_foot, mass 0.5; collision box size=0.05 0.1 0.2; visual box size=0.05 0.1 0.2
- added link player6_x
- added link player6_y
Joints:
- added joint player5_joint: type continuous, parent player5_y, child player5, origin xyz=0.03 0 0.3, axis 0 0 1
- added joint player5_left_foot_joint: type revolute, parent player5, child player5_left_foot, origin xyz=0.10 0.06 0, axis 0 -1 0
- added joint player5_right_foot_joint: type revolute, parent player5, child player5_right_foot, origin xyz=0.10 -0.06 0, axis 0 -1 0
- added joint player5_x_joint: type prismatic, parent field, child player5_x, axis 1 0 0
- added joint player5_y_joint: type prismatic, parent player5_x, child player5_y, axis 0 1 0
- added joint player6_joint: type continuous, parent player6_y, child player6, origin xyz=0.03 0 0.3, axis 0 0 1
- added joint player6_left_foot_joint: type revolute, parent player6, child player6_left_foot, origin xyz=0.10 0.06 0, axis 0 -1 0
- added joint player6_right_foot_joint: type revolute, parent player6, child player6_right_foot, origin xyz=0.10 -0.06 0, axis 0 -1 0
- added joint player6_x_joint: type prismatic, parent field, child player6_x, axis 1 0 0
- added joint player6_y_joint: type prismatic, parent player6_x, child player6_y, axis 0 1 0

File: assets/soccer_robot.xacro (robot description, xacro)
@@ -9,5 +9,7 @@
   <xacro:player name="player1" color="blue"/>
   <xacro:player name="player2" color="blue"/>
-  <xacro:player name="player3" color="red"/>
+  <xacro:player name="player3" color="blue"/>
   <xacro:player name="player4" color="red"/>
+  <xacro:player name="player5" color="red"/>
+  <xacro:player name="player6" color="red"/>
 </robot>

Commit message: refine model

File: assets/soccer.urdf (robot description, URDF)
Before this commit: robot soccer, 42 links, 41 joints
Links:
- link player1: geometry collision box size=0.130 0.200 0.600; visual box size=0.130 0.200 0.600
- link player1_left_foot: geometry collision box size=0.020 0.100 0.240; visual box size=0.020 0.090 0.240
- link player1_right_foot: geometry collision box size=0.020 0.100 0.240; visual box size=0.020 0.090 0.240
- link player2: geometry collision box size=0.130 0.200 0.600; visual box size=0.130 0.200 0.600
- link player2_left_foot: geometry collision box size=0.020 0.100 0.240; visual box size=0.020 0.090 0.240
- link player2_right_foot: geometry collision box size=0.020 0.100 0.240; visual box size=0.020 0.090 0.240
- link player3: geometry collision box size=0.130 0.200 0.600; visual box size=0.130 0.200 0.600
- link player3_left_foot: geometry collision box size=0.020 0.100 0.240; visual box size=0.020 0.090 0.240
- link player3_right_foot: geometry collision box size=0.020 0.100 0.240; visual box size=0.020 0.090 0.240
- link player4: geometry collision box size=0.130 0.200 0.600; visual box size=0.130 0.200 0.600
- link player4_left_foot: geometry collision box size=0.020 0.100 0.240; visual box size=0.020 0.090 0.240
- link player4_right_foot: geometry collision box size=0.020 0.100 0.240; visual box size=0.020 0.090 0.240
- link player5: geometry collision box size=0.130 0.200 0.600; visual box size=0.130 0.200 0.600
- link player5_left_foot: geometry collision box size=0.020 0.100 0.240; visual box size=0.020 0.090 0.240
- link player5_right_foot: geometry collision box size=0.020 0.100 0.240; visual box size=0.020 0.090 0.240
- link player6: geometry collision box size=0.130 0.200 0.600; visual box size=0.130 0.200 0.600
- link player6_left_foot: geometry collision box size=0.020 0.100 0.240; visual box size=0.020 0.090 0.240
- link player6_right_foot: geometry collision box size=0.020 0.100 0.240; visual box size=0.020 0.090 0.240
Joints:
- joint player1_joint: origin xyz=0.03 0 0.3 -> (none)
- joint player1_left_foot_joint: origin xyz=0.10 0.06 0 -> xyz=0.070 0.055 0.250
- joint player1_right_foot_joint: origin xyz=0.10 -0.06 0 -> xyz=0.070 -0.055 0.250
- joint player2_joint: origin xyz=0.03 0 0.3 -> (none)
- joint player2_left_foot_joint: origin xyz=0.10 0.06 0 -> xyz=0.070 0.055 0.250
- joint player2_right_foot_joint: origin xyz=0.10 -0.06 0 -> xyz=0.070 -0.055 0.250
- joint player3_joint: origin xyz=0.03 0 0.3 -> (none)
- joint player3_left_foot_joint: origin xyz=0.10 0.06 0 -> xyz=0.070 0.055 0.250
- joint player3_right_foot_joint: origin xyz=0.10 -0.06 0 -> xyz=0.070 -0.055 0.250
- joint player4_joint: origin xyz=0.03 0 0.3 -> (none)
- joint player4_left_foot_joint: origin xyz=0.10 0.06 0 -> xyz=0.070 0.055 0.250
- joint player4_right_foot_joint: origin xyz=0.10 -0.06 0 -> xyz=0.070 -0.055 0.250
- joint player5_joint: origin xyz=0.03 0 0.3 -> (none)
- joint player5_left_foot_joint: origin xyz=0.10 0.06 0 -> xyz=0.070 0.055 0.250
- joint player5_right_foot_joint: origin xyz=0.10 -0.06 0 -> xyz=0.070 -0.055 0.250
- joint player6_joint: origin xyz=0.03 0 0.3 -> (none)
- joint player6_left_foot_joint: origin xyz=0.10 0.06 0 -> xyz=0.070 0.055 0.250
- joint player6_right_foot_joint: origin xyz=0.10 -0.06 0 -> xyz=0.070 -0.055 0.250

Commit message: fix foot size

File: assets/soccer.urdf (robot description, URDF)
Before this commit: robot soccer, 42 links, 41 joints
Links:
- link player1_left_foot: geometry collision box size=0.020 0.090 0.240; visual box size=0.020 0.090 0.240
- link player1_right_foot: geometry collision box size=0.020 0.090 0.240; visual box size=0.020 0.090 0.240
- link player2_left_foot: geometry collision box size=0.020 0.090 0.240; visual box size=0.020 0.090 0.240
- link player2_right_foot: geometry collision box size=0.020 0.090 0.240; visual box size=0.020 0.090 0.240
- link player3_left_foot: geometry collision box size=0.020 0.090 0.240; visual box size=0.020 0.090 0.240
- link player3_right_foot: geometry collision box size=0.020 0.090 0.240; visual box size=0.020 0.090 0.240
- link player4_left_foot: geometry collision box size=0.020 0.090 0.240; visual box size=0.020 0.090 0.240
- link player4_right_foot: geometry collision box size=0.020 0.090 0.240; visual box size=0.020 0.090 0.240
- link player5_left_foot: geometry collision box size=0.020 0.090 0.240; visual box size=0.020 0.090 0.240
- link player5_right_foot: geometry collision box size=0.020 0.090 0.240; visual box size=0.020 0.090 0.240
- link player6_left_foot: geometry collision box size=0.020 0.090 0.240; visual box size=0.020 0.090 0.240
- link player6_right_foot: geometry collision box size=0.020 0.090 0.240; visual box size=0.020 0.090 0.240
